Commit message: Add files via upload

File: assets/ur5/lw_ur_description/urdf/ur10.urdf.xacro (robot description, xacro)
@@ -5,6 +5,6 @@
   Contributers: Jimmy Da Silva, Ajit Krisshna N L, Muhammad Asif Rana
 -->
-  <xacro:include filename="$(find lw_ur_description)/urdf/ur.transmission.xacro" />
-  <xacro:include filename="$(find lw_ur_description)/urdf/ur.gazebo.xacro" />
+  <xacro:include filename="$(find liwei_ur_description)/urdf/ur.transmission.xacro" />
+  <xacro:include filename="$(find liwei_ur_description)/urdf/ur.gazebo.xacro" />
   <xacro:macro name="cylinder_inertial" params="radius length mass *origin">
     <inertial>
@@ -50,5 +50,5 @@
     <xacro:property name="elbow_offset" value="0.049042" /> <!-- measured from model -->
     <xacro:property name="upper_arm_inertia_offset" value="0.175" />  <!-- measured from model -->
-    <!-- This is for compatibility reasons, as transformation between base and base_link was always 180 degree in the lw_ur_description -->
+    <!-- This is for compatibility reasons, as transformation between base and base_link was always 180 degree in the liwei_ur_description -->
     <xacro:property name="base_correction" value="${pi}" />
     <link name="${prefix}base_link" >
@@ -56,5 +56,5 @@
         <origin xyz="0 0 0" rpy="0 0 ${base_correction}"/>
         <geometry>
-          <mesh filename="package://lw_ur_description/meshes/ur10/visual/base.dae"/>
+          <mesh filename="package://liwei_ur_description/meshes/ur10/visual/base.dae"/>
         </geometry>
         <material name="LightGrey">
@@ -65,5 +65,5 @@
         <origin xyz="0 0 0" rpy="0 0 ${base_correction}"/>
         <geometry>
-          <mesh filename="package://lw_ur_description/meshes/ur10/collision/base.stl"/>
+          <mesh filename="package://liwei_ur_description/meshes/ur10/collision/base.stl"/>
         </geometry>
       </collision>
@@ -95,5 +95,5 @@
         <origin xyz="0 0 0" rpy="0 0 ${pi}"/>
         <geometry>
-          <mesh filename="package://lw_ur_description/meshes/ur10/visual/shoulder.dae"/>
+          <mesh filename="package://liwei_ur_description/meshes/ur10/visual/shoulder.dae"/>
         </geometry>
         <material name="LightGrey">
@@ -104,5 +104,5 @@
         <origin xyz="0 0 0" rpy="0 0 ${pi}"/>
         <geometry>
-          <mesh filename="package://lw_ur_description/meshes/ur10/collision/shoulder.stl"/>
+          <mesh filename="package://liwei_ur_description/meshes/ur10/collision/shoulder.stl"/>
         </geometry>
       </collision>
@@ -134,5 +134,5 @@
         <origin xyz="0 0 ${shoulder_offset}" rpy="${pi/2} 0 ${-pi/2}"/>
         <geometry>
-          <mesh filename="package://lw_ur_description/meshes/ur10/visual/upperarm.dae"/>
+          <mesh filename="package://liwei_ur_description/meshes/ur10/visual/upperarm.dae"/>
         </geometry>
         <material name="LightGrey">
@@ -143,5 +143,5 @@
         <origin xyz="0 0 ${shoulder_offset}" rpy="${pi/2} 0 ${-pi/2}"/>
         <geometry>
-          <mesh filename="package://lw_ur_description/meshes/ur10/collision/upperarm.stl"/>
+          <mesh filename="package://liwei_ur_description/meshes/ur10/collision/upperarm.stl"/>
         </geometry>
       </collision>
@@ -173,5 +173,5 @@
         <origin xyz="0 0 ${elbow_offset}" rpy="${pi/2} 0 ${-pi/2}"/>
         <geometry>
-          <mesh filename="package://lw_ur_description/meshes/ur10/visual/forearm.dae"/>
+          <mesh filename="package://liwei_ur_description/meshes/ur10/visual/forearm.dae"/>
         </geometry>
         <material name="LightGrey">
@@ -182,5 +182,5 @@
         <origin xyz="0 0 ${elbow_offset}" rpy="${pi/2} 0 ${-pi/2}"/>
         <geometry>
-          <mesh filename="package://lw_ur_description/meshes/ur10/collision/forearm.stl"/>
+          <mesh filename="package://liwei_ur_description/meshes/ur10/collision/forearm.stl"/>
         </geometry>
       </collision>
@@ -212,5 +212,5 @@
         <origin xyz="0 0 -0.1149" rpy="${pi/2} 0 0"/>
         <geometry>
-          <mesh filename="package://lw_ur_description/meshes/ur10/visual/wrist1.dae"/>
+          <mesh filename="package://liwei_ur_description/meshes/ur10/visual/wrist1.dae"/>
         </geometry>
         <material name="LightGrey">
@@ -221,5 +221,5 @@
         <origin xyz="0 0 -0.1149" rpy="${pi/2} 0 0"/>
         <geometry>
-          <mesh filename="package://lw_ur_description/meshes/ur10/collision/wrist1.stl"/>
+          <mesh filename="package://liwei_ur_description/meshes/ur10/collision/wrist1.stl"/>
         </geometry>
       </collision>
@@ -251,5 +251,5 @@
         <origin xyz="0 0 -0.1158" rpy="0 0 0"/>
         <geometry>
-          <mesh filename="package://lw_ur_description/meshes/ur10/visual/wrist2.dae"/>
+          <mesh filename="package://liwei_ur_description/meshes/ur10/visual/wrist2.dae"/>
         </geometry>
         <material name="LightGrey">
@@ -260,5 +260,5 @@
         <origin xyz="0 0 -0.1158" rpy="0 0 0"/>
         <geometry>
-          <mesh filename="package://lw_ur_description/meshes/ur10/collision/wrist2.stl"/>
+          <mesh filename="package://liwei_ur_description/meshes/ur10/collision/wrist2.stl"/>
         </geometry>
       </collision>
@@ -290,5 +290,5 @@
         <origin xyz="0 0 -0.0922" rpy="${pi/2} 0 0"/>
         <geometry>
-          <mesh filename="package://lw_ur_description/meshes/ur10/visual/wrist3.dae"/>
+          <mesh filename="package://liwei_ur_description/meshes/ur10/visual/wrist3.dae"/>
         </geometry>
         <material name="LightGrey">
@@ -299,5 +299,5 @@
         <origin xyz="0 0 -0.0922" rpy="${pi/2} 0 0"/>
         <geometry>
-          <mesh filename="package://lw_ur_description/meshes/ur10/collision/wrist3.stl"/>
+          <mesh filename="package://liwei_ur_description/meshes/ur10/collision/wrist3.stl"/>
         </geometry>
       </collision>

File: assets/ur5/lw_ur_description/urdf/ur10_kong.urdf.xacro (robot description, xacro)
@@ -5,6 +5,6 @@
   Contributers: Jimmy Da Silva, Ajit Krisshna N L, Muhammad Asif Rana
 -->
-  <xacro:include filename="$(find lw_ur_description)/urdf/ur.transmission.xacro" />
-  <xacro:include filename="$(find lw_ur_description)/urdf/ur.gazebo.xacro" />
+  <xacro:include filename="$(find liwei_ur_description)/urdf/ur.transmission.xacro" />
+  <xacro:include filename="$(find liwei_ur_description)/urdf/ur.gazebo.xacro" />
   <xacro:macro name="cylinder_inertial" params="radius length mass *origin">
     <inertial>
@@ -16,5 +16,5 @@
     </inertial>
   </xacro:macro>
-  <xacro:macro name="ur10_robot" params="prefix joint_limited
+  <xacro:macro name="ur10_robot_kong" params="prefix joint_limited
     shoulder_pan_lower_limit:=${-pi}    shoulder_pan_upper_limit:=${pi}
     shoulder_lift_lower_limit:=${-pi}    shoulder_lift_upper_limit:=${pi}
@@ -50,5 +50,5 @@
     <xacro:property name="elbow_offset" value="0.049042" /> <!-- measured from model -->
     <xacro:property name="upper_arm_inertia_offset" value="0.175" />  <!-- measured from model -->
-    <!-- This is for compatibility reasons, as transformation between base and base_link was always 180 degree in the lw_ur_description -->
+    <!-- This is for compatibility reasons, as transformation between base and base_link was always 180 degree in the liwei_ur_description -->
     <xacro:property name="base_correction" value="${pi}" />
     <link name="${prefix}base_link" >
@@ -56,5 +56,5 @@
         <origin xyz="0 0 0" rpy="0 0 ${base_correction}"/>
         <geometry>
-          <mesh filename="package://lw_ur_description/meshes/ur10/visual/base.dae"/>
+          <mesh filename="package://liwei_ur_description/meshes/ur10/visual/base.dae"/>
         </geometry>
         <material name="LightGrey">
@@ -65,5 +65,5 @@
         <origin xyz="0 0 0" rpy="0 0 ${base_correction}"/>
         <geometry>
-          <mesh filename="package://lw_ur_description/meshes/ur10/collision/base.stl"/>
+          <mesh filename="package://liwei_ur_description/meshes/ur10/collision/base.stl"/>
         </geometry>
       </collision>
@@ -95,5 +95,5 @@
         <origin xyz="0 0 0" rpy="0 0 ${pi}"/>
         <geometry>
-          <mesh filename="package://lw_ur_description/meshes/ur10/visual/shoulder.dae"/>
+          <mesh filename="package://liwei_ur_description/meshes/ur10/visual/shoulder.dae"/>
         </geometry>
         <material name="LightGrey">
@@ -104,5 +104,5 @@
         <origin xyz="0 0 0" rpy="0 0 ${pi}"/>
         <geometry>
-          <mesh filename="package://lw_ur_description/meshes/ur10/collision/shoulder.stl"/>
+          <mesh filename="package://liwei_ur_description/meshes/ur10/collision/shoulder.stl"/>
         </geometry>
       </collision>
@@ -134,5 +134,5 @@
         <origin xyz="0 0 ${shoulder_offset}" rpy="${pi/2} 0 ${-pi/2}"/>
         <geometry>
-          <mesh filename="package://lw_ur_description/meshes/ur10/visual/upperarm.dae"/>
+          <mesh filename="package://liwei_ur_description/meshes/ur10/visual/upperarm.dae"/>
         </geometry>
         <material name="LightGrey">
@@ -143,5 +143,5 @@
         <origin xyz="0 0 ${shoulder_offset}" rpy="${pi/2} 0 ${-pi/2}"/>
         <geometry>
-          <mesh filename="package://lw_ur_description/meshes/ur10/collision/upperarm.stl"/>
+          <mesh filename="package://liwei_ur_description/meshes/ur10/collision/upperarm.stl"/>
         </geometry>
       </collision>
@@ -173,5 +173,5 @@
         <origin xyz="0 0 ${elbow_offset}" rpy="${pi/2} 0 ${-pi/2}"/>
         <geometry>
-          <mesh filename="package://lw_ur_description/meshes/ur10/visual/forearm.dae"/>
+          <mesh filename="package://liwei_ur_description/meshes/ur10/visual/forearm.dae"/>
         </geometry>
         <material name="LightGrey">
@@ -182,5 +182,5 @@
         <origin xyz="0 0 ${elbow_offset}" rpy="${pi/2} 0 ${-pi/2}"/>
         <geometry>
-          <mesh filename="package://lw_ur_description/meshes/ur10/collision/forearm.stl"/>
+          <mesh filename="package://liwei_ur_description/meshes/ur10/collision/forearm.stl"/>
         </geometry>
       </collision>
@@ -212,5 +212,5 @@
         <origin xyz="0 0 -0.1149" rpy="${pi/2} 0 0"/>
         <geometry>
-          <mesh filename="package://lw_ur_description/meshes/ur10/visual/wrist1.dae"/>
+          <mesh filename="package://liwei_ur_description/meshes/ur10/visual/wrist1.dae"/>
         </geometry>
         <material name="LightGrey">
@@ -221,5 +221,5 @@
         <origin xyz="0 0 -0.1149" rpy="${pi/2} 0 0"/>
         <geometry>
-          <mesh filename="package://lw_ur_description/meshes/ur10/collision/wrist1.stl"/>
+          <mesh filename="package://liwei_ur_description/meshes/ur10/collision/wrist1.stl"/>
         </geometry>
       </collision>
@@ -251,5 +251,5 @@
         <origin xyz="0 0 -0.1158" rpy="0 0 0"/>
         <geometry>
-          <mesh filename="package://lw_ur_description/meshes/ur10/visual/wrist2.dae"/>
+          <mesh filename="package://liwei_ur_description/meshes/ur10/visual/wrist2.dae"/>
         </geometry>
         <material name="LightGrey">
@@ -260,5 +260,5 @@
         <origin xyz="0 0 -0.1158" rpy="0 0 0"/>
         <geometry>
-          <mesh filename="package://lw_ur_description/meshes/ur10/collision/wrist2.stl"/>
+          <mesh filename="package://liwei_ur_description/meshes/ur10/collision/wrist2.stl"/>
         </geometry>
       </collision>
@@ -290,5 +290,5 @@
         <origin xyz="0 0 -0.0922" rpy="${pi/2} 0 0"/>
         <geometry>
-          <mesh filename="package://lw_ur_description/meshes/ur10/visual/wrist3.dae"/>
+          <mesh filename="package://liwei_ur_description/meshes/ur10/visual/wrist3.dae"/>
         </geometry>
         <material name="LightGrey">
@@ -299,5 +299,5 @@
         <origin xyz="0 0 -0.0922" rpy="${pi/2} 0 0"/>
         <geometry>
-          <mesh filename="package://lw_ur_description/meshes/ur10/collision/wrist3.stl"/>
+          <mesh filename="package://liwei_ur_description/meshes/ur10/collision/wrist3.stl"/>
         </geometry>
       </collision>

File: assets/ur5/lw_ur_description/urdf/ur10_robot.urdf.xacro (robot description, xacro)
@@ -3,8 +3,8 @@
     <xacro:arg name="transmission_hw_interface" default="hardware_interface/PositionJointInterface"/>
     <!-- common stuff -->
-    <xacro:include filename="$(find lw_ur_description)/urdf/common.gazebo.xacro" />
+    <xacro:include filename="$(find liwei_ur_description)/urdf/common.gazebo.xacro" />
     <!-- ur10 -->
-    <xacro:include filename="$(find lw_ur_description)/urdf/ur10.urdf.xacro" />
-    <xacro:include filename="$(find lw_ur_description)/urdf/ur10_kong.urdf.xacro" />
+    <xacro:include filename="$(find liwei_ur_description)/urdf/ur10.urdf.xacro" />
+    <xacro:include filename="$(find liwei_ur_description)/urdf/ur10_kong.urdf.xacro" />
     <xacro:include filename="$(find dual_description)/urdf/soft_hybrid_gripper_URDF.urdf" />
     <xacro:include filename="$(find dual_description)/urdf/soft_hybrid_gripper2_URDF.urdf" />
@@ -13,5 +13,5 @@
     <xacro:include filename="$(find dual_description)/urdf/robot_optical_table_kong.urdf" />
     <!-- arm -->
-    <xacro:arg name="kinematics_config" default="$(find lw_ur_description)/config/ur10_default.yaml"/>
+    <xacro:arg name="kinematics_config" default="$(find liwei_ur_description)/config/ur10_default.yaml"/>
     <xacro:ur10_robot prefix="hong_" joint_limited="false"
     shoulder_pan_lower_limit="${-2*pi}" shoulder_pan_upper_limit="${2*pi}"
@@ -23,5 +23,5 @@
     transmission_hw_interface="$(arg transmission_hw_interface)"
     kinematics_file="${load_yaml('$(arg kinematics_config)')}" />
-    <xacro:arg name="kinematics_config_kong" default="$(find lw_ur_description)/config/ur10_default.yaml"/>
+    <xacro:arg name="kinematics_config_kong" default="$(find liwei_ur_description)/config/ur10_default.yaml"/>
     <xacro:ur10_robot_kong prefix="kong_" joint_limited="false"
     shoulder_pan_lower_limit="${-2*pi}" shoulder_pan_upper_limit="${2*pi}"

File: assets/ur5/lw_ur_description/urdf/ur10_soft_and_robotiq.xacro (robot description, xacro)
@@ -3,15 +3,17 @@
     <xacro:arg name="transmission_hw_interface" default="hardware_interface/PositionJointInterface"/>
     <!-- common stuff -->
-    <xacro:include filename="$(find lw_ur_description)/urdf/common.gazebo.xacro" />
+    <xacro:include filename="$(find liwei_ur_description)/urdf/common.gazebo.xacro" />
     <!-- ur10 -->
-    <xacro:include filename="$(find lw_ur_description)/urdf/ur10.urdf.xacro" />
-    <xacro:include filename="$(find lw_ur_description)/urdf/ur10_kong.urdf.xacro" />
+    <xacro:include filename="$(find liwei_ur_description)/urdf/ur10.urdf.xacro" />
+    <xacro:include filename="$(find liwei_ur_description)/urdf/ur10_kong.urdf.xacro" />
+    <xacro:include filename="$(find robotiq_ft_sensor)/urdf/robotiq_fts150.urdf.xacro" />
+    <xacro:include filename="$(find robotiq_2f_140_gripper_visualization)/urdf/robotiq_arg2f_140_model_macro.xacro" />
+    <!--<xacro:include filename="$(find dual_description)/urdf/soft_gripper_urdf.urdf" />-->
     <xacro:include filename="$(find dual_description)/urdf/soft_hybrid_gripper_URDF.urdf" />
-    <xacro:include filename="$(find dual_description)/urdf/soft_hybrid_gripper2_URDF.urdf" />
     <xacro:include filename="$(find dual_description)/urdf/robot_movable_table.urdf" />
     <xacro:include filename="$(find dual_description)/urdf/robot_optical_table_hong.urdf" />
     <xacro:include filename="$(find dual_description)/urdf/robot_optical_table_kong.urdf" />
     <!-- arm -->
-    <xacro:arg name="kinematics_config" default="$(find lw_ur_description)/config/ur10_default.yaml"/>
+    <xacro:arg name="kinematics_config" default="$(find liwei_ur_description)/config/ur10_default.yaml"/>
     <xacro:ur10_robot prefix="hong_" joint_limited="false"
     shoulder_pan_lower_limit="${-2*pi}" shoulder_pan_upper_limit="${2*pi}"
@@ -23,5 +25,5 @@
     transmission_hw_interface="$(arg transmission_hw_interface)"
     kinematics_file="${load_yaml('$(arg kinematics_config)')}" />
-    <xacro:arg name="kinematics_config_kong" default="$(find lw_ur_description)/config/ur10_default.yaml"/>
+    <xacro:arg name="kinematics_config_kong" default="$(find liwei_ur_description)/config/ur10_default.yaml"/>
     <xacro:ur10_robot_kong prefix="kong_" joint_limited="false"
     shoulder_pan_lower_limit="${-2*pi}" shoulder_pan_upper_limit="${2*pi}"
@@ -33,14 +35,20 @@
     transmission_hw_interface="$(arg transmission_hw_interface)"
     kinematics_file="${load_yaml('$(arg kinematics_config_kong)')}" />
+    <!-- force torque sensor -->
+    <xacro:robotiq_fts150 prefix="" parent="hong_tool0" >
+      <origin xyz="0 0 0" rpy="0 0 0"/>
+    </xacro:robotiq_fts150>
+    <!-- robotiq_arg2f_140 -->
+    <xacro:robotiq_arg2f_140 prefix=""/>
+    <joint name="ft_gripper_joint" type="fixed">
+     <parent link="robotiq_ft_frame_id"/>
+     <child link="robotiq_arg2f_base_link"/>
+     <origin xyz="0 0 0" rpy="0 0 0"/>
+    </joint>
     <!-- soft gripper -->
-    <joint name="soft_robot_joint_kong" type="fixed">
-        <parent link="kong_tool0"/>
-        <child link="base_link2"/>
-        <origin xyz="0 0 0" rpy="0 0 ${pi}"/>
-    </joint>
-    <joint name="soft_robot_joint_hong" type="fixed">
-        <parent link="hong_tool0"/>
-        <child link="base_link1"/>
-        <origin xyz="0 0 0" rpy="0 0 ${pi}"/>
+    <joint name="soft_robot_joint" type="fixed">
+     <parent link="kong_tool0"/>
+     <child link="base_link1"/>
+     <origin xyz="0 0 0" rpy="0 0 ${pi}"/>
     </joint>
     <!--environment-->
@@ -54,20 +62,20 @@
         <parent link="world" />
         <child link="robot_optical_table_hong" />
-        <origin xyz="1.35 0.012 0.016" rpy="0 0 ${pi}" />
+        <origin xyz="-1.35 0 0" rpy="0 0 0" />
     </joint>
     <joint name="world_to_optical_table_kong" type="fixed">
         <parent link="world" />
         <child link="robot_optical_table_kong" />
-        <origin xyz="-1.381 0 0" rpy="0 0 ${pi}" />
+        <origin xyz="1.35 0 0" rpy="0 0 0" />
     </joint>
     <joint name="optical_table_to_hong" type="fixed">
         <parent link="robot_optical_table_hong" />
         <child link = "hong_base_link" />
-        <origin xyz="0.465 0 0.77" rpy="0.0 0.0 ${-pi/2}" />
+        <origin xyz="0.465 0 0.77" rpy="0.0 0.0 ${pi/2}" />
     </joint>
     <joint name="optical_table_to_kong" type="fixed">
         <parent link="robot_optical_table_kong" />
         <child link = "kong_base_link" />
-        <origin xyz="-0.465 0 0.77" rpy="0.0 0.0 ${pi/2}" />
+        <origin xyz="-0.465 0 0.77" rpy="0.0 0.0 ${-pi/2}" />
     </joint>
 </robot>

File: assets/ur5/ur10.urdf (robot description, URDF)
Before this commit: robot ur10, 8 links, 7 joints
Links:
- link base_link: geometry collision mesh filename=package://lw_ur_description/meshes/ur10/collision/base.stl; visual mesh filename=package://lw_ur_description/meshes/ur10/visual/base.dae
- link forearm_link: geometry collision mesh filename=package://lw_ur_description/meshes/ur10/collision/forearm.s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; visual mesh filename=package://lw_ur_description/meshes/ur10/visual/forearm.dae
- link shoulder_link: geometry collision mesh filename=package://lw_ur_description/meshes/ur10/collision/shoulder.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; visual mesh filename=package://lw_ur_description/meshes/ur10/visual/shoulder.dae
- link upper_arm_link: geometry collision mesh filename=package://lw_ur_description/meshes/ur10/collision/upperarm.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; visual mesh filename=package://lw_ur_description/meshes/ur10/visual/upperarm.dae
- link wrist_1_link: geometry collision mesh filename=package://lw_ur_description/meshes/ur10/collision/wrist1.stl; visual mesh filename=package://lw_ur_description/meshes/ur10/visual/wrist1.dae
- link wrist_2_link: geometry collision mesh filename=package://lw_ur_description/meshes/ur10/collision/wrist2.stl; visual mesh filename=package://lw_ur_description/meshes/ur10/visual/wrist2.dae
- link wrist_3_link: geometry collision mesh filename=package://lw_ur_description/meshes/ur10/collision/wrist3.stl; visual mesh filename=package://lw_ur_description/meshes/ur10/visual/wrist3.dae

File: assets/ur5/ur10_hong_gripper.urdf (robot description, URDF)
Before this commit: robot , 12 links, 11 joints
Links:
- link base_link: geometry collision mesh filename=assets/ur5/lw_ur_description/meshes/ur10/collision/base.stl scale=1.00000 1.00000 1.00000; visual mesh filename=assets/ur5/lw_ur_description/meshes/ur10/visual/base.dae scale=1.00000 1.00000 1.00000
- link forearm_link: geometry collision mesh filename=assets/ur5/lw_ur_description/meshes/ur10/collision/forearm.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 scale=1.00000 1.00000 1.00000; visual mesh filename=assets/ur5/lw_ur_description/meshes/ur10/visual/forearm.dae scale=1.00000 1.00000 1.00000
- link shoulder_link: geometry collision mesh filename=assets/ur5/lw_ur_description/meshes/ur10/collision/shoulder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 scale=1.00000 1.00000 1.00000; visual mesh filename=assets/ur5/lw_ur_description/meshes/ur10/visual/shoulder.dae scale=1.00000 1.00000 1.00000
- link upper_arm_link: geometry collision mesh filename=assets/ur5/lw_ur_description/meshes/ur10/collision/upperarm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 scale=1.00000 1.00000 1.00000; visual mesh filename=assets/ur5/lw_ur_description/meshes/ur10/visual/upperarm.dae scale=1.00000 1.00000 1.00000
- link wrist_1_link: geometry collision mesh filename=assets/ur5/lw_ur_description/meshes/ur10/collision/wrist1.s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 scale=1.00000 1.00000 1.00000; visual mesh filename=assets/ur5/lw_ur_description/meshes/ur10/visual/wrist1.dae scale=1.00000 1.00000 1.00000
- link wrist_2_link: geometry collision mesh filename=assets/ur5/lw_ur_description/meshes/ur10/collision/wrist2.s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 scale=1.00000 1.00000 1.00000; visual mesh filename=assets/ur5/lw_ur_description/meshes/ur10/visual/wrist2.dae scale=1.00000 1.00000 1.00000
- link wrist_3_link: geometry collision mesh filename=assets/ur5/lw_ur_description/meshes/ur10/collision/wrist3.s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 scale=1.00000 1.00000 1.00000; visual mesh filename=assets/ur5/lw_ur_description/meshes/ur10/visual/wrist3.dae scale=1.00000 1.00000 1.00000
