Commit message: Add files via upload

File: assets/ur5/ur10_kong.urdf (robot description, URDF)
Before this commit: robot ur10_kong, 8 links, 7 joints
Links:
- link kong_base_link: geometry collision mesh filename=package://lw_ur_description/meshes/ur10/collision/base.stl; visual mesh filename=package://lw_ur_description/meshes/ur10/visual/base.dae
- link kong_forearm_link: geometry collision mesh filename=package://lw_ur_description/meshes/ur10/collision/forearm.s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; visual mesh filename=package://lw_ur_description/meshes/ur10/visual/forearm.dae
- link kong_shoulder_link: geometry collision mesh filename=package://lw_ur_description/meshes/ur10/collision/shoulder.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; visual mesh filename=package://lw_ur_description/meshes/ur10/visual/shoulder.dae
- link kong_upper_arm_link: geometry collision mesh filename=package://lw_ur_description/meshes/ur10/collision/upperarm.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; visual mesh filename=package://lw_ur_description/meshes/ur10/visual/upperarm.dae
- link kong_wrist_1_link: geometry collision mesh filename=package://lw_ur_description/meshes/ur10/collision/wrist1.stl; visual mesh filename=package://lw_ur_description/meshes/ur10/visual/wrist1.dae
- link kong_wrist_2_link: geometry collision mesh filename=package://lw_ur_description/meshes/ur10/collision/wrist2.stl; visual mesh filename=package://lw_ur_description/meshes/ur10/visual/wrist2.dae
- link kong_wrist_3_link: geometry collision mesh filename=package://lw_ur_description/meshes/ur10/collision/wrist3.stl; visual mesh filename=package://lw_ur_description/meshes/ur10/visual/wrist3.dae

File: assets/ur5/ur10_kong_gripper.urdf (robot description, URDF)
Before this commit: robot , 12 links, 11 joints
Links:
- link kong_base_link: geometry collision mesh filename=assets/ur5/lw_ur_description/meshes/ur10/collision/base.stl scale=1.00000 1.00000 1.00000; visual mesh filename=assets/ur5/lw_ur_description/meshes/ur10/visual/base.dae scale=1.00000 1.00000 1.00000
- link kong_forearm_link: geometry collision mesh filename=assets/ur5/lw_ur_description/meshes/ur10/collision/forearm.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 scale=1.00000 1.00000 1.00000; visual mesh filename=assets/ur5/lw_ur_description/meshes/ur10/visual/forearm.dae scale=1.00000 1.00000 1.00000
- link kong_shoulder_link: geometry collision mesh filename=assets/ur5/lw_ur_description/meshes/ur10/collision/shoulder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 scale=1.00000 1.00000 1.00000; visual mesh filename=assets/ur5/lw_ur_description/meshes/ur10/visual/shoulder.dae scale=1.00000 1.00000 1.00000
- link kong_upper_arm_link: geometry collision mesh filename=assets/ur5/lw_ur_description/meshes/ur10/collision/upperarm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 scale=1.00000 1.00000 1.00000; visual mesh filename=assets/ur5/lw_ur_description/meshes/ur10/visual/upperarm.dae scale=1.00000 1.00000 1.00000
- link kong_wrist_1_link: geometry collision mesh filename=assets/ur5/lw_ur_description/meshes/ur10/collision/wrist1.s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 scale=1.00000 1.00000 1.00000; visual mesh filename=assets/ur5/lw_ur_description/meshes/ur10/visual/wrist1.dae scale=1.00000 1.00000 1.00000
- link kong_wrist_2_link: geometry collision mesh filename=assets/ur5/lw_ur_description/meshes/ur10/collision/wrist2.s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 scale=1.00000 1.00000 1.00000; visual mesh filename=assets/ur5/lw_ur_description/meshes/ur10/visual/wrist2.dae scale=1.00000 1.00000 1.00000
- link kong_wrist_3_link: geometry collision mesh filename=assets/ur5/lw_ur_description/meshes/ur10/collision/wrist3.s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 scale=1.00000 1.00000 1.00000; visual mesh filename=assets/ur5/lw_ur_description/meshes/ur10/visual/wrist3.dae scale=1.00000 1.00000 1.00000
