Commit message: Add files via upload

File: assets/ur5/soft_hybrid_gripper_URDF.urdf (robot description, URDF)
Before this commit: robot soft hybrid gripper URDF, 4 links, 3 joints
Links:
- link base_link1: geometry collision mesh filename=collision/base_link_cam.STL; visual mesh filename=collision/base_link_cam.STL

File: assets/ur5/ur10_hong_gripper.urdf (robot description, URDF)
Before this commit: robot , 12 links, 11 joints
Links:
- link base_link1: geometry collision mesh filename=assets/ur5/collision/base_link_cam.STL scale=1.00000 1.00000 1.00000; visual mesh filename=assets/ur5/collision/base_link_cam.STL scale=1.00000 1.00000 1.00000
Joints:
- joint rigid_rev_joint1: origin xyz=-0.01800 0.06040 0.03100 rpy=0.00000 -0.00000 0.00000 -> xyz=-0.01800 0.06040 0.03100 rpy=0.00000 -0.76 0.00000

File: assets/ur5/ur10_hong_gripper_cam.urdf (robot description, URDF)
Before this commit: robot , 12 links, 11 joints
Links:
- removed link base_link2
- removed link kong_base_link
- removed link kong_ee_link
- removed link kong_forearm_link
- removed link kong_shoulder_link
- removed link kong_upper_arm_link
- removed link kong_wrist_1_link
- removed link kong_wrist_2_link
- removed link kong_wrist_3_link
- removed link rigid_link2
- removed link rigid_tip_link2
- removed link soft_tip_link2
- added link base_link, mass 4.00000; collision mesh filename=assets/ur5/lw_ur_description/meshes/ur10/collision/base.stl scale=1.00000 1.00000 1.00000; visual mesh filename=assets/ur5/lw_ur_description/meshes/ur10/visual/base.dae scale=1.00000 1.00000 1.00000
- added link base_link1, mass 0.11784; collision mesh filename=assets/ur5/collision/base_link_cam.STL scale=1.00000 1.00000 1.00000; visual mesh filename=assets/ur5/collision/base_link_cam.STL scale=1.00000 1.00000 1.00000
- added link ee_link, mass 1.00000
- added link forearm_link, mass 3.87000; collision mesh filename=assets/ur5/lw_ur_description/meshes/ur10/collision/forearm.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 scale=1.00000 1.00000 1.00000; visual mesh filename=assets/ur5/lw_ur_description/meshes/ur10/visual/forearm.dae scale=1.00000 1.00000 1.00000
- added link rigid_link1, mass 0.04453; collision mesh filename=assets/ur5/collision/rigid_link.STL scale=1.00000 1.00000 1.00000; visual mesh filename=assets/ur5/collision/rigid_link.STL scale=1.00000 1.00000 1.00000
- added link rigid_tip_link1, mass 0.01345; collision mesh filename=assets/ur5/collision/rigid_tip_link.STL scale=1.00000 1.00000 1.00000; visual mesh filename=assets/ur5/collision/rigid_tip_link.STL scale=1.00000 1.00000 1.00000
- added link shoulder_link, mass 7.77800; collision mesh filename=assets/ur5/lw_ur_description/meshes/ur10/collision/shoulder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 scale=1.00000 1.00000 1.00000; visual mesh filename=assets/ur5/lw_ur_description/meshes/ur10/visual/shoulder.dae scale=1.00000 1.00000 1.00000
- added link soft_tip_link1, mass 0.02675; collision mesh filename=assets/ur5/collision/soft_tip_link.STL scale=1.00000 1.00000 1.00000; visual mesh filename=assets/ur5/collision/soft_tip_link.STL scale=1.00000 1.00000 1.00000
- added link upper_arm_link, mass 12.93000; collision mesh filename=assets/ur5/lw_ur_description/meshes/ur10/collision/upperarm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 scale=1.00000 1.00000 1.00000; visual mesh filename=assets/ur5/lw_ur_description/meshes/ur10/visual/upperarm.dae scale=1.00000 1.00000 1.00000
- added link wrist_1_link, mass 1.96000; collision mesh filename=assets/ur5/lw_ur_description/meshes/ur10/collision/wrist1.s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 scale=1.00000 1.00000 1.00000; visual mesh filename=assets/ur5/lw_ur_description/meshes/ur10/visual/wrist1.dae scale=1.00000 1.00000 1.00000
- added link wrist_2_link, mass 1.96000; collision mesh filename=assets/ur5/lw_ur_description/meshes/ur10/collision/wrist2.s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 scale=1.00000 1.00000 1.00000; visual mesh filename=assets/ur5/lw_ur_description/meshes/ur10/visual/wrist2.dae scale=1.00000 1.00000 1.00000
- added link wrist_3_link, mass 0.20200; collision mesh filename=assets/ur5/lw_ur_description/meshes/ur10/collision/wrist3.s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 scale=1.00000 1.00000 1.00000; visual mesh filename=assets/ur5/lw_ur_description/meshes/ur10/visual/wrist3.dae scale=1.00000 1.00000 1.00000
Joints:
- removed joint kong_ee_fixed_joint
- removed joint kong_elbow_joint
- removed joint kong_shoulder_lift_joint
- removed joint kong_shoulder_pan_joint
- removed joint kong_wrist_1_joint
- removed joint kong_wrist_2_joint
- removed joint kong_wrist_3_joint
- removed joint rigid_rev_joint2
- removed joint rigid_tip_joint2
- removed joint soft_tip_joint2
- added joint ee_fixed_joint: type fixed, parent wrist_3_link, child ee_link, origin xyz=0.00000 0.09220 0.00000 rpy=0.00000 -0.00000 1.57080, axis 0.00000 0.00000 0.00000
- added joint elbow_joint: type revolute, parent upper_arm_link, child forearm_link, origin xyz=0.00000 -0.17190 0.61200 rpy=0.00000 -0.00000 0.00000, axis 0.00000 1.00000 0.00000, limit lower=-6.2831853 upper=6.2831853 effort=150.0 velocity=3.15
- added joint rigid_rev_joint1: type revolute, parent base_link1, child rigid_link1, origin xyz=-0.01800 0.06040 0.03100 rpy=0.00000 -0.00000 0.00000, axis 0.00000 -1.00000 0.00000, limit lower=-3.1415926 upper=3.1415926 effort=0 velocity=0
- added joint rigid_tip_joint1: type fixed, parent rigid_link1, child rigid_tip_link1, origin xyz=0.02939 -0.00085 0.11906 rpy=0.00000 -0.13252 3.14159, axis 0.00000 0.00000 0.00000
- added joint shoulder_lift_joint: type revolute, parent shoulder_link, child upper_arm_link, origin xyz=0.00000 0.22094 0.00000 rpy=0.00000 1.57080 -0.00000, axis 0.00000 1.00000 0.00000, limit lower=-6.2831853 upper=6.2831853 effort=330.0 velocity=2.16
- added joint shoulder_pan_joint: type revolute, parent base_link, child shoulder_link, origin xyz=0.00000 0.00000 0.12730 rpy=0.00000 -0.00000 0.00000, axis 0.00000 0.00000 1.00000, limit lower=-6.2831853 upper=6.2831853 effort=330.0 velocity=2.16
- added joint soft_tip_joint1: type fixed, parent base_link1, child soft_tip_link1, origin xyz=0.11681 0.06100 0.09874 rpy=0.00000 -0.66549 0.00000, axis 0.00000 0.00000 0.00000
- added joint wrist_1_joint: type revolute, parent forearm_link, child wrist_1_link, origin xyz=0.00000 0.00000 0.57230 rpy=0.00000 1.57080 -0.00000, axis 0.00000 1.00000 0.00000, limit lower=-6.2831853 upper=6.2831853 effort=54.0 velocity=3.2
- added joint wrist_2_joint: type revolute, parent wrist_1_link, child wrist_2_link, origin xyz=0.00000 0.11490 0.00000 rpy=0.00000 -0.00000 0.00000, axis 0.00000 0.00000 1.00000, limit lower=-6.2831853 upper=6.2831853 effort=54.0 velocity=3.2
- added joint wrist_3_joint: type revolute, parent wrist_2_link, child wrist_3_link, origin xyz=0.00000 0.00000 0.11570 rpy=0.00000 -0.00000 0.00000, axis 0.00000 1.00000 0.00000, limit lower=-6.2831853 upper=6.2831853 effort=54.0 velocity=3.2
- joint joint_dummy1: child base_link2 -> base_link1; parent kong_ee_link -> ee_link
