Commit message: Add files via upload

File: assets/ur5/liwei_ur_description/urdf/ur10.urdf.xacro (robot description, xacro)
@@ -17,10 +17,10 @@
   </xacro:macro>
   <xacro:macro name="ur10_robot" params="prefix joint_limited
-    shoulder_pan_lower_limit:=${-pi}    shoulder_pan_upper_limit:=${pi}
-    shoulder_lift_lower_limit:=${-pi}    shoulder_lift_upper_limit:=${pi}
-    elbow_joint_lower_limit:=${-pi}    elbow_joint_upper_limit:=${pi}
-    wrist_1_lower_limit:=${-pi}    wrist_1_upper_limit:=${pi}
-    wrist_2_lower_limit:=${-pi}    wrist_2_upper_limit:=${pi}
-    wrist_3_lower_limit:=${-pi}    wrist_3_upper_limit:=${pi}
+    shoulder_pan_lower_limit:=${-2*pi}    shoulder_pan_upper_limit:=${2*pi}
+    shoulder_lift_lower_limit:=${-2*pi}    shoulder_lift_upper_limit:=${2*pi}
+    elbow_joint_lower_limit:=${-2*pi}    elbow_joint_upper_limit:=${2*pi}
+    wrist_1_lower_limit:=${-2*pi}    wrist_1_upper_limit:=${2*pi}
+    wrist_2_lower_limit:=${-2*pi}    wrist_2_upper_limit:=${2*pi}
+    wrist_3_lower_limit:=${-2*pi}    wrist_3_upper_limit:=${2*pi}
     transmission_hw_interface:=hardware_interface/PositionJointInterface
     safety_limits:=false safety_pos_margin:=0.15
@@ -50,5 +50,5 @@
     <xacro:property name="elbow_offset" value="0.049042" /> <!-- measured from model -->
     <xacro:property name="upper_arm_inertia_offset" value="0.175" />  <!-- measured from model -->
-    <!-- This is for compatibility reasons, as transformation between base and base_link was always 180 degree in the liwei_ur_description -->
+    <!-- This is for compatibility reasons, as transformation between base and base_link was always 180 degree in the ur_description -->
     <xacro:property name="base_correction" value="${pi}" />
     <link name="${prefix}base_link" >

File: assets/ur5/liwei_ur_description/urdf/ur10_kong.urdf.xacro (robot description, xacro)
@@ -17,10 +17,10 @@
   </xacro:macro>
   <xacro:macro name="ur10_robot_kong" params="prefix joint_limited
-    shoulder_pan_lower_limit:=${-pi}    shoulder_pan_upper_limit:=${pi}
-    shoulder_lift_lower_limit:=${-pi}    shoulder_lift_upper_limit:=${pi}
-    elbow_joint_lower_limit:=${-pi}    elbow_joint_upper_limit:=${pi}
-    wrist_1_lower_limit:=${-pi}    wrist_1_upper_limit:=${pi}
-    wrist_2_lower_limit:=${-pi}    wrist_2_upper_limit:=${pi}
-    wrist_3_lower_limit:=${-pi}    wrist_3_upper_limit:=${pi}
+    shoulder_pan_lower_limit:=${-2*pi}    shoulder_pan_upper_limit:=${2*pi}
+    shoulder_lift_lower_limit:=${-2*pi}    shoulder_lift_upper_limit:=${2*pi}
+    elbow_joint_lower_limit:=${-2*pi}    elbow_joint_upper_limit:=${2*pi}
+    wrist_1_lower_limit:=${-2*pi}    wrist_1_upper_limit:=${2*pi}
+    wrist_2_lower_limit:=${-2*pi}    wrist_2_upper_limit:=${2*pi}
+    wrist_3_lower_limit:=${-2*pi}    wrist_3_upper_limit:=${2*pi}
     transmission_hw_interface:=hardware_interface/PositionJointInterface
     safety_limits:=false safety_pos_margin:=0.15
@@ -50,5 +50,5 @@
     <xacro:property name="elbow_offset" value="0.049042" /> <!-- measured from model -->
     <xacro:property name="upper_arm_inertia_offset" value="0.175" />  <!-- measured from model -->
-    <!-- This is for compatibility reasons, as transformation between base and base_link was always 180 degree in the liwei_ur_description -->
+    <!-- This is for compatibility reasons, as transformation between base and base_link was always 180 degree in the ur_description -->
     <xacro:property name="base_correction" value="${pi}" />
     <link name="${prefix}base_link" >
@@ -56,5 +56,5 @@
         <origin xyz="0 0 0" rpy="0 0 ${base_correction}"/>
         <geometry>
-          <mesh filename="package://liwei_ur_description/meshes/ur10/visual/base.dae"/>
+          <mesh filename="package://ur_description/meshes/ur10/visual/base.dae"/>
         </geometry>
         <material name="LightGrey">
@@ -65,5 +65,5 @@
         <origin xyz="0 0 0" rpy="0 0 ${base_correction}"/>
         <geometry>
-          <mesh filename="package://liwei_ur_description/meshes/ur10/collision/base.stl"/>
+          <mesh filename="package://ur_description/meshes/ur10/collision/base.stl"/>
         </geometry>
       </collision>
@@ -95,5 +95,5 @@
         <origin xyz="0 0 0" rpy="0 0 ${pi}"/>
         <geometry>
-          <mesh filename="package://liwei_ur_description/meshes/ur10/visual/shoulder.dae"/>
+          <mesh filename="package://ur_description/meshes/ur10/visual/shoulder.dae"/>
         </geometry>
         <material name="LightGrey">
@@ -104,5 +104,5 @@
         <origin xyz="0 0 0" rpy="0 0 ${pi}"/>
         <geometry>
-          <mesh filename="package://liwei_ur_description/meshes/ur10/collision/shoulder.stl"/>
+          <mesh filename="package://ur_description/meshes/ur10/collision/shoulder.stl"/>
         </geometry>
       </collision>
@@ -134,5 +134,5 @@
         <origin xyz="0 0 ${shoulder_offset}" rpy="${pi/2} 0 ${-pi/2}"/>
         <geometry>
-          <mesh filename="package://liwei_ur_description/meshes/ur10/visual/upperarm.dae"/>
+          <mesh filename="package://ur_description/meshes/ur10/visual/upperarm.dae"/>
         </geometry>
         <material name="LightGrey">
@@ -143,5 +143,5 @@
         <origin xyz="0 0 ${shoulder_offset}" rpy="${pi/2} 0 ${-pi/2}"/>
         <geometry>
-          <mesh filename="package://liwei_ur_description/meshes/ur10/collision/upperarm.stl"/>
+          <mesh filename="package://ur_description/meshes/ur10/collision/upperarm.stl"/>
         </geometry>
       </collision>
@@ -173,5 +173,5 @@
         <origin xyz="0 0 ${elbow_offset}" rpy="${pi/2} 0 ${-pi/2}"/>
         <geometry>
-          <mesh filename="package://liwei_ur_description/meshes/ur10/visual/forearm.dae"/>
+          <mesh filename="package://ur_description/meshes/ur10/visual/forearm.dae"/>
         </geometry>
         <material name="LightGrey">
@@ -182,5 +182,5 @@
         <origin xyz="0 0 ${elbow_offset}" rpy="${pi/2} 0 ${-pi/2}"/>
         <geometry>
-          <mesh filename="package://liwei_ur_description/meshes/ur10/collision/forearm.stl"/>
+          <mesh filename="package://ur_description/meshes/ur10/collision/forearm.stl"/>
         </geometry>
       </collision>
@@ -212,5 +212,5 @@
         <origin xyz="0 0 -0.1149" rpy="${pi/2} 0 0"/>
         <geometry>
-          <mesh filename="package://liwei_ur_description/meshes/ur10/visual/wrist1.dae"/>
+          <mesh filename="package://ur_description/meshes/ur10/visual/wrist1.dae"/>
         </geometry>
         <material name="LightGrey">
@@ -221,5 +221,5 @@
         <origin xyz="0 0 -0.1149" rpy="${pi/2} 0 0"/>
         <geometry>
-          <mesh filename="package://liwei_ur_description/meshes/ur10/collision/wrist1.stl"/>
+          <mesh filename="package://ur_description/meshes/ur10/collision/wrist1.stl"/>
         </geometry>
       </collision>
@@ -251,5 +251,5 @@
         <origin xyz="0 0 -0.1158" rpy="0 0 0"/>
         <geometry>
-          <mesh filename="package://liwei_ur_description/meshes/ur10/visual/wrist2.dae"/>
+          <mesh filename="package://ur_description/meshes/ur10/visual/wrist2.dae"/>
         </geometry>
         <material name="LightGrey">
@@ -260,5 +260,5 @@
         <origin xyz="0 0 -0.1158" rpy="0 0 0"/>
         <geometry>
-          <mesh filename="package://liwei_ur_description/meshes/ur10/collision/wrist2.stl"/>
+          <mesh filename="package://ur_description/meshes/ur10/collision/wrist2.stl"/>
         </geometry>
       </collision>
@@ -290,5 +290,5 @@
         <origin xyz="0 0 -0.0922" rpy="${pi/2} 0 0"/>
         <geometry>
-          <mesh filename="package://liwei_ur_description/meshes/ur10/visual/wrist3.dae"/>
+          <mesh filename="package://ur_description/meshes/ur10/visual/wrist3.dae"/>
         </geometry>
         <material name="LightGrey">
@@ -299,5 +299,5 @@
         <origin xyz="0 0 -0.0922" rpy="${pi/2} 0 0"/>
         <geometry>
-          <mesh filename="package://liwei_ur_description/meshes/ur10/collision/wrist3.stl"/>
+          <mesh filename="package://ur_description/meshes/ur10/collision/wrist3.stl"/>
         </geometry>
       </collision>

File: assets/ur5/liwei_ur_description/urdf/ur10_robot.urdf.xacro (robot description, xacro)
@@ -7,6 +7,6 @@
     <xacro:include filename="$(find liwei_ur_description)/urdf/ur10.urdf.xacro" />
     <xacro:include filename="$(find liwei_ur_description)/urdf/ur10_kong.urdf.xacro" />
-    <xacro:include filename="$(find dual_description)/urdf/soft_hybrid_gripper_URDF.urdf" />
-    <xacro:include filename="$(find dual_description)/urdf/soft_hybrid_gripper2_URDF.urdf" />
+    <xacro:include filename="$(find hybrid_griper_v3)/urdf/hybrid_griper_v3.urdf" />
+    <xacro:include filename="$(find rigid_fixture)/urdf/rigid_fixture.urdf" />
     <xacro:include filename="$(find dual_description)/urdf/robot_movable_table.urdf" />
     <xacro:include filename="$(find dual_description)/urdf/robot_optical_table_hong.urdf" />
@@ -36,11 +36,11 @@
     <joint name="soft_robot_joint_kong" type="fixed">
         <parent link="kong_tool0"/>
-        <child link="base_link2"/>
-        <origin xyz="0 0 0" rpy="0 0 ${pi}"/>
+        <child link="base_link1"/>
+        <origin xyz="0 0 0" rpy="0 0 ${pi/2}"/>
     </joint>
     <joint name="soft_robot_joint_hong" type="fixed">
         <parent link="hong_tool0"/>
-        <child link="base_link1"/>
-        <origin xyz="0 0 0" rpy="0 0 ${pi}"/>
+        <child link="base_link"/>
+        <origin xyz="0 0 0" rpy="0 0 ${-pi}"/>
     </joint>
     <!--environment-->
